File: 2019-Pi-Power.kicad_pcb (KiCad board)
At the start: 2 copper layers, 65 x 56 mm, 132 parts, among them J1 Barrel_Jack_Switch, J2 USB_A, J3 USB_A, J4 Conn_02x04_Odd_Even, J5 Conn_01x04, J6 Conn_01x04, J7 Conn_01x04, J8 Conn_02x02_Odd_Even, P1 Conn_02x20_Odd_Even, U1 MP1584

Commit message: V1 of DSKY-matic variant of this board
Parts:
- removed 0 (x105): SolderWirePad_single_0-8mmDrill, Wire_Pads:SolderWirePad_single_0-8mmDrill
- removed the J7 at (211.1, 102.4)
- removed the REF** at (220.1, 147.7)
- removed REF***: OSHW-Logo_5.7x6mm_SilkScreen, Symbols:OSHW-Logo_5.7x6mm_SilkScreen
- added C10: 220pF, Capacitor_SMD:C_0603_1608Metric, F.Cu at (241.4, 113.7)
- added C6: 100nF, Capacitor_SMD:C_0603_1608Metric, F.Cu at (246.5, 123.1)
- added C7: 10uF, Capacitor_SMD:C_Elec_6.3x5.8, F.Cu at (239.4, 130.9)
- added C8: 100nF, Capacitor_SMD:C_0603_1608Metric, F.Cu at (243.4, 125.9)
- added C9: 22uF, Capacitor_SMD:C_Elec_6.3x5.8, F.Cu at (255.9, 126.9)
- added D2: D_Schottky, digikey-footprints:DO-214AC, F.Cu at (249.5, 123.3)
- added L2: 10uH, Inductor_SMD:L_10.4x10.4_H4.8, F.Cu at (252.0, 113.4)
- added R5: 124K, Resistor_SMD:R_0603_1608Metric, F.Cu at (235.3, 116.0)
- added R6: 40.2k, Resistor_SMD:R_0603_1608Metric, F.Cu at (237.6, 115.2)
- added R7: 200k, Resistor_SMD:R_0603_1608Metric, F.Cu at (239.1, 125.9)
- added R8: 68.1k, Resistor_SMD:R_0603_1608Metric, F.Cu at (239.9, 113.7)
- added REF**: OSHW-Logo2_7.3x6mm_SilkScreen, Symbol:OSHW-Logo2_7.3x6mm_SilkScreen, F.Cu at (236.6, 145.7)
- added U2: MP1584, Package_SO:SO-8_5.3x6.2mm_P1.27mm, F.Cu at (241.9, 120.3)
- C1: renamed from C3; footprint Capacitors_SMD:C_0603 -> Capacitor_SMD:C_0603_1608Metric
- C2: renamed from C1; footprint Capacitors_SMD:CP_Elec_6.3x5.8 -> Capacitor_SMD:C_Elec_6.3x5.8
- C3: renamed from C2; footprint Capacitors_SMD:C_0603 -> Capacitor_SMD:C_0603_1608Metric
- C4: renamed from C5; footprint Capacitors_SMD:CP_Elec_6.3x5.8 -> Capacitor_SMD:C_Elec_6.3x5.8
- D1: footprint Digikey:DO-214AC -> digikey-footprints:DO-214AC
- J2, J3: value USB_A -> Conn_01x04; footprint USB_A:61400416021 -> Connector_PinHeader_2.54mm:PinHeader_1x04_P2.54mm_Vertical
- L1: value 15uH -> 22uH; footprint Inductors_SMD:L_10.4x10.4_H4.8 -> Inductor_SMD:L_10.4x10.4_H4.8
- R1: renamed from R4; footprint Resistors_SMD:R_0603 -> Resistor_SMD:R_0603_1608Metric
- R2: footprint Resistors_SMD:R_0603 -> Resistor_SMD:R_0603_1608Metric
- R3: renamed from R1; footprint Resistors_SMD:R_0603 -> Resistor_SMD:R_0603_1608Metric
- R4: renamed from R3; footprint Resistors_SMD:R_0603 -> Resistor_SMD:R_0603_1608Metric
- U1: footprint Housings_SOIC:SOIC-8_3.9x4.9mm_Pitch1.27mm -> Package_SO:SO-8_5.3x6.2mm_P1.27mm
- moved J2 54.7 mm to (208.4, 103.5)
- moved C2 21.8 mm to (212.4, 130.9), turned to 180 degrees
- moved C4 18.3 mm to (228.4, 127.4), turned to 270 degrees
- moved R3 17.4 mm to (212.4, 125.9)
- moved C3 17.4 mm to (215.7, 125.9)
- moved R1 17.3 mm to (207.9, 115.7)
- moved L1 17.2 mm to (223.9, 113.7), turned to 180 degrees
- moved C5 17.1 mm to (213.6, 113.4)
- moved U1 17.1 mm to (214.3, 120.2)
- moved R4 17.1 mm to (211.9, 113.4)
- moved R2 17.0 mm to (210.2, 114.9)
- moved D1 16.9 mm to (222.6, 123.3)
- moved C1 16.7 mm to (219.3, 123.1)
- moved J1 9.67 mm to (227.4, 138.1)
- moved J4 7.24 mm to (241.9, 144.2)
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- renumbered C4 to C5, J8 to J7, MK3 to MK2, MK2 to MK3
Connections:
- J1 pad 3: Net-(J1-Pad3) -> (no net)
- J2 pad 2: Net-(J2-Pad2) -> /GPIO2(SDA1)
- J2 pad 3: Net-(J2-Pad3) -> /GPIO3(SCL1)
- J3 pad 1: +5V -> /+3.3V_SUPP
- J3 pad 2: Net-(J3-Pad2) -> /+3.3V_SUPP
- J3 pad 3: Net-(J3-Pad3) -> GND
- P1 pad 10: /GPIO15(RXD0) -> (no net)
- P1 pad 11: /GPIO17(GEN0) -> (no net)
- P1 pad 12: /GPIO18(GEN1)(PWM0) -> (no net)
- P1 pad 13: /GPIO27(GEN2) -> (no net)
- P1 pad 15: /GPIO22(GEN3) -> (no net)
- P1 pad 16: /GPIO23(GEN4) -> (no net)
- P1 pad 18: /GPIO24(GEN5) -> (no net)
- P1 pad 22: /GPIO25(GEN6) -> (no net)
- P1 pad 27: /ID_SD -> (no net)
- P1 pad 28: /ID_SC -> (no net)
- P1 pad 29: /GPIO5 -> (no net)
- P1 pad 31: /GPIO6 -> (no net)
- P1 pad 32: /GPIO12(PWM0) -> (no net)
- P1 pad 33: /GPIO13(PWM1) -> (no net)
- P1 pad 35: /GPIO19(SPI1_MISO) -> (no net)
- P1 pad 36: /GPIO16 -> (no net)
- P1 pad 37: /GPIO26 -> (no net)
- P1 pad 38: /GPIO20(SPI1_MOSI) -> (no net)
- P1 pad 40: /GPIO21(SPI1_SCK) -> (no net)
- P1 pad 7: /GPIO4(GCLK) -> (no net)
- P1 pad 8: /GPIO14(TXD0) -> (no net)
- U1 pad 2: VCC_EN -> (no net)
Routing:
- net /+3.3V_SUPP: track 0.00 -> 48.1 mm, vias 0 -> 2
- net Net-(C2-Pad1): track 3.30 -> 47.7 mm
- net GND: track 0.00 -> 32.0 mm, vias 26 -> 124
- net +3V3: track 6.98 -> 24.2 mm
- net +5V: track 95.1 -> 87.3 mm, vias 8 -> 3
- net Net-(C6-Pad1): track 0.00 -> 5.41 mm
- net Net-(R5-Pad2): track 0.00 -> 4.29 mm
- net Net-(R7-Pad1): track 0.00 -> 2.94 mm
- net Net-(C6-Pad2): track 0.00 -> 2.69 mm
- net Net-(C10-Pad1): track 0.00 -> 2.37 mm
- net Net-(C10-Pad2): track 0.00 -> 1.52 mm
- net Net-(R3-Pad1): track 3.88 -> 2.40 mm
- net /GPIO9(SPI0_MISO): track 6.15 -> 7.31 mm
- net /GPIO11(SPI0_SCK): track 6.15 -> 7.31 mm
- net /GPIO10(SPI0_MOSI): track 6.15 -> 7.31 mm
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- added copper zone on B.Cu, net /+3.3V_SUPP
- added copper zone on F.Cu, net /+3.3V_SUPP
- added copper zone on F.Cu, net Net-(C6-Pad1)
- removed copper zone on F.Cu, net Net-(C2-Pad1)
Other:
- outline, holes or cut-outs redrawn
- rule via_min_drill: 0.5 -> 0.3
- rule via_min_size: 0.8 -> 0.3
- board text added: "+3.3V"
- board text added: "DSKY-matic Pi Power V1 Riley Rainey https://github.com/rrainey/DSKY-matic"
- board text added: "GND"
- board text added: "RASPBERRY-PI 40-PIN ADDON BOARD VIEW FROM TOP NOTE: P1 SHOULD BE FITTED ON THE REVERSE OF THE BOARD"
- board text removed: "CAMERA"
- board text removed: "Electricgraveyard.com"
- board text removed: "RASPBERRY-PI 40-PIN ADDON BOARD VIEW FROM TOP NOTE: P1 SHOULD BE FITTED ON THE REVERSE OF THE BOARD ADD EDGE CUTS FROM CAMERA AND DISPLAY PORTS AS REQUIRED"
