File: 2019-Pi-Power.sch (KiCad schematic (older format))
At the start: 25 parts, among them J1 Barrel_Jack_Switch, J2 USB_A, J3 USB_A, J4 Conn_02x04_Odd_Even, J5 Conn_01x04, J6 Conn_01x04, J7 Conn_01x04, J8 Conn_02x02_Odd_Even, P1 Conn_02x20_Odd_Even, U1 MP1584

Commit message: V1 of DSKY-matic variant of this board
Parts:
- removed J2, J3: USB_A, USB_A:61400416021, symbol Connector:USB_A
- removed J7: Conn_01x04, Pin_Headers:Pin_Header_Straight_1x04_Pitch2.54mm, symbol Connector_Generic:Conn_01x04
- added C10: 220pF, Capacitor_SMD:C_0603_1608Metric, symbol Device:C
- added C6, C8: 100nF, Capacitor_SMD:C_0603_1608Metric, symbol Device:C
- added C7: 10uF, Capacitor_SMD:C_Elec_6.3x5.8, symbol Device:C
- added C9: 22uF, Capacitor_SMD:C_Elec_6.3x5.8, symbol Device:C
- added D2: D_Schottky, digikey-footprints:DO-214AC, symbol dk_Diodes-Rectifiers-Single:B340A-13-F
- added J2, J3: Conn_01x04, Connector_PinHeader_2.54mm:PinHeader_1x04_P2.54mm_Vertical, symbol Connector_Generic:Conn_01x04
- added L2: 10uH, Inductor_SMD:L_10.4x10.4_H4.8, symbol Device:L
- added R5: 124K, Resistor_SMD:R_0603_1608Metric, symbol Device:R
- added R6: 40.2k, Resistor_SMD:R_0603_1608Metric, symbol Device:R
- added R7: 200k, Resistor_SMD:R_0603_1608Metric, symbol Device:R
- added R8: 68.1k, Resistor_SMD:R_0603_1608Metric, symbol Device:R
- added U2: MP1584, Package_SO:SO-8_5.3x6.2mm_P1.27mm, symbol Pi-Power:Monolithic_Power_MP1584
- C1: renamed from C3; footprint Capacitors_SMD:C_0603 -> Capacitor_SMD:C_0603_1608Metric
- C2: renamed from C1; footprint Capacitors_SMD:CP_Elec_6.3x5.8 -> Capacitor_SMD:C_Elec_6.3x5.8
- C3: renamed from C2; footprint Capacitors_SMD:C_0603 -> Capacitor_SMD:C_0603_1608Metric
- C4: renamed from C5; footprint Capacitors_SMD:CP_Elec_6.3x5.8 -> Capacitor_SMD:C_Elec_6.3x5.8
- D1: footprint Digikey:DO-214AC -> digikey-footprints:DO-214AC
- L1: footprint Inductors_SMD:L_10.4x10.4_H4.8 -> Inductor_SMD:L_10.4x10.4_H4.8
- R1: renamed from R4; footprint Resistors_SMD:R_0603 -> Resistor_SMD:R_0603_1608Metric
- R2: footprint Resistors_SMD:R_0603 -> Resistor_SMD:R_0603_1608Metric
- R3: renamed from R1; footprint Resistors_SMD:R_0603 -> Resistor_SMD:R_0603_1608Metric
- R4: renamed from R3; footprint Resistors_SMD:R_0603 -> Resistor_SMD:R_0603_1608Metric
- U1: footprint Housings_SOIC:SO-8_5.3x6.2mm_Pitch1.27mm -> Package_SO:SO-8_5.3x6.2mm_P1.27mm; symbol Monolithic_Power:MP1584 -> Pi-Power:Monolithic_Power_MP1584
- renumbered C4 to C5, J8 to J7, MK3 to MK2, MK2 to MK3
Connections:
- net labels added: +3.3V_SUPP
- net labels removed: VCC_EN
- wire segments 131 -> 157
- no-connect marks 0 -> 2
Other:
- moved on the sheet: J4, J5, J6, J7
