File: 2019-Pi-Power.kicad_sch (KiCad schematic)
At the start: 36 parts, among them J1 Barrel_Jack_Switch, J2 1719710004, J3 Conn_01x04, J4 Conn_02x04_Odd_Even, J5 Conn_01x04, J6 Conn_01x04, J7 Conn_02x02_Odd_Even, P1 Conn_02x20_Odd_Even, U1 MP1584, U2 MP1584

Commit message: V4 PCB
Parts:
- C1, C3, C6, C8: MANUFACTURER (none) -> Samsung; MPN (none) -> CL10B104KB8NNNC
- C10: MANUFACTURER (none) -> Samsung; MPN (none) -> CL10B221KB8NFNC
- C2, C7: MANUFACTURER (none) -> Panasonic; MPN (none) -> EEE-1HA100SP
- C4, C9: MANUFACTURER (none) -> Panasonic; MPN (none) -> EEH-ZA1H220P
- C5: MANUFACTURER (none) -> Samsung; MPN (none) -> CL10B151KB8NNNC
- D1, D2: MANUFACTURER (none) -> Diodes Incorporated; MPN (none) -> B340A-13-F
- J1: MANUFACTURER (none) -> Same Sky (formerly CUI); MPN (none) -> PJ-002AH
- J2: MPN (none) -> 1719710004; now not fitted
- J4, J5, J6, J7: now not fitted
- L1: MANUFACTURER (none) -> Würth Elektronik; MPN (none) -> 7447714220
- L2: MANUFACTURER (none) -> Würth Elektronik; MPN (none) -> 744065100
- MK1, MK2, MK3, MK4: now left out of the parts list
- R1: MANUFACTURER (none) -> Panasonic; MPN (none) -> ERJ-H3EF2103V
- R2, R6: MANUFACTURER (none) -> Panasonic; MPN (none) -> ERA-3VEB4022V
- R3, R4: MANUFACTURER (none) -> Panasonic; MPN (none) -> ERJ-H3EF1003V
- R5: MANUFACTURER (none) -> KOA; MPN (none) -> RN73R1JTTD1243D25
- R7: MANUFACTURER (none) -> Panasonic; MPN (none) -> ERJ-H3EF2003V
- R8: MANUFACTURER (none) -> Vishay; MPN (none) -> MCT06030C6812FP500
- U1, U2: MANUFACTURER (none) -> Monolithic Power; MPN (none) -> MP1584EN-LF-Z
